File: UccMicroDuino/UccMicroDuino.kicad_pcb (KiCad board)
At the start: 2 copper layers, 8 parts, among them J1 Conn_01x10_Socket, J2 USB_A, U1 ATtiny85-20S

Commit message: Add files via upload
Parts:
- added D3: 3.6V 1/2mW, Diode_SMD:D_SOD-123, F.Cu at (207.3, 65.0)
- added D4: LED, ledSmd:ledSMD, F.Cu at (196.0, 80.0)
- added R2: 68Ω 5% 1/8W, Resistor_SMD:R_0805_2012Metric_Pad1.20x1.40mm_HandSolder, F.Cu at (199.0, 67.0)
- added R3: 68Ω 5% 1/8W, Resistor_SMD:R_0805_2012Metric_Pad1.20x1.40mm_HandSolder, F.Cu at (206.0, 60.0)
- added R4: 330Ω 5% 1/8W, Resistor_SMD:R_0805_2012Metric_Pad1.20x1.40mm_HandSolder, F.Cu at (187.0, 78.0)
- added R5: R, Resistor_SMD:R_0805_2012Metric_Pad1.20x1.40mm_HandSolder, F.Cu at (180.0, 72.0)
- C1: value C -> 0.1u
- D1: value D_Filled -> PMLL 4148L
- D2: value D_Zener -> 3.6V 1/2mW
- PcbUSBTypeA1: renamed from J2; value USB_A -> PMLL 4148L
- R1: value R -> 1.5KΩ 5% 1/8W
- moved U1 73.3 mm to (205.0, 80.0), turned to 180 degrees
- moved J1 59.9 mm to (180.9, 87.0), turned to 90 degrees
- moved D2 59.3 mm to (185.0, 70.3), turned to -90 degrees
- moved R1 54.5 mm to (193.0, 67.0), turned to 90 degrees
- moved D1 52.0 mm to (175.0, 62.0), turned to 90 degrees
- moved PcbUSBTypeA1 47.9 mm to (175.5, 52.2), turned to -90 degrees
- moved D5 42.7 mm to (177.0, 77.0), turned to 180 degrees
- moved C1 39.4 mm to (178.0, 69.0), turned to 180 degrees
- renumbered D3 to D5
Connections:
- C1 pad 1: unconnected-(C1-Pad1) -> +5V
- C1 pad 2: unconnected-(C1-Pad2) -> GND
- D1 pad 2: unconnected-(D1-A-Pad2) -> Net-(D1-A)
- D2 pad 1: unconnected-(D2-K-Pad1) -> Net-(D2-K)
- D2 pad 2: unconnected-(D2-A-Pad2) -> GND
- D5 pad 1: unconnected-(D3-K-Pad1) -> Net-(D5-K)
- D5 pad 2: unconnected-(D3-A-Pad2) -> +5V
- J1 pad 1: unconnected-(J1-Pin_1-Pad1) -> +5V
- J1 pad 2: unconnected-(J1-Pin_2-Pad2) -> GND
- J1 pad 4: unconnected-(J1-Pin_4-Pad4) -> Net-(J1-Pin_4)
- J1 pad 5: unconnected-(J1-Pin_5-Pad5) -> Net-(D4-A)
- J1 pad 6: unconnected-(J1-Pin_6-Pad6) -> Net-(J1-Pin_6)
- J1 pad 7: unconnected-(J1-Pin_7-Pad7) -> Net-(J1-Pin_7)
- J1 pad 8: unconnected-(J1-Pin_8-Pad8) -> Net-(J1-Pin_8)
- J1 pad 9: unconnected-(J1-Pin_9-Pad9) -> Net-(J1-Pin_9)
- PcbUSBTypeA1 pad 1: unconnected-(J2-VBUS-Pad1) -> Net-(D1-A)
- PcbUSBTypeA1 pad 2: unconnected-(J2-D--Pad2) -> Net-(D2-K)
- PcbUSBTypeA1 pad 3: unconnected-(J2-D+-Pad3) -> Net-(D3-K)
- PcbUSBTypeA1 pad 4: unconnected-(J2-GND-Pad4) -> GND
- R1 pad 2: unconnected-(R1-Pad2) -> Net-(D2-K)
- U1 pad 1: unconnected-(U1-~{RESET}/PB5-Pad1) -> Net-(J1-Pin_9)
- U1 pad 2: unconnected-(U1-XTAL1/PB3-Pad2) -> Net-(J1-Pin_7)
- U1 pad 3: unconnected-(U1-XTAL2/PB4-Pad3) -> Net-(J1-Pin_8)
- U1 pad 4: unconnected-(U1-GND-Pad4) -> GND
- U1 pad 5: unconnected-(U1-AREF/PB0-Pad5) -> Net-(J1-Pin_4)
- U1 pad 6: unconnected-(U1-PB1-Pad6) -> Net-(D4-A)
- U1 pad 7: unconnected-(U1-PB2-Pad7) -> Net-(J1-Pin_6)
- U1 pad 8: unconnected-(U1-VCC-Pad8) -> +5V
Routing:
- net GND: track 0.00 -> 167.0 mm
- net +5V: track 0.00 -> 72.2 mm
- net Net-(J1-Pin_8): track 0.00 -> 47.1 mm
- net Net-(D3-K): track 0.00 -> 38.5 mm
- net Net-(D2-K): track 0.00 -> 38.4 mm
- net Net-(J1-Pin_7): track 0.00 -> 31.3 mm
- net Net-(J1-Pin_4): track 0.00 -> 17.8 mm
- net Net-(D4-A): track 0.00 -> 14.2 mm
- net Net-(J1-Pin_6): track 0.00 -> 10.7 mm
- net Net-(J1-Pin_9): track 0.00 -> 9.52 mm
- net Net-(D1-A): track 0.00 -> 9.49 mm
- net Net-(D4-K): track 0.00 -> 7.03 mm
- net Net-(D5-K): track 0.00 -> 5.08 mm
Other:
- board outline added: 45 x 45 mm
